File: je03-pcb-guide.kicad_pcb (KiCad board)
At the start: 2 copper layers, 69.8 x 38.1 mm, 24 parts, among them SW1 SW_Push, U1 ATmega32U4-AU, Y1 16MHz

Commit message: Organize file
Routing:
- added copper zone on B.Cu, net GND
Other:
- board text added: "Jack Esche"
Changed lines of the file:
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@@
   (general
     (thickness 1.6)
-    (drawings 8)
+    (drawings 9)
     (tracks 259)
     (zones 0)
@@
       (rotate (xyz 0 0 0))
     )
+  )
+  (gr_text "Jack Esche" (at 117.221 114.935) (layer F.Cu)
+    (effects (font (size 1.5 1.5) (thickness 0.3)))
   )
   (gr_line (start 123.825 117.475) (end 57.15 117.475) (layer Edge.Cuts) (width 0.05))
@@
   (segment (start 62.357 91.821) (end 63.119 92.456) (width 0.254) (layer B.Cu) (net 19))
   (segment (start 83.566 102.392) (end 81.691 102.392) (width 0.254) (layer B.Cu) (net 20))
+  (zone (net 1) (net_name GND) (layer B.Cu) (hatch edge 0.508)
+    (connect_pads (clearance 0.508))
+    (min_thickness 0.254)
+    (fill yes (arc_segments 32) (thermal_gap 0.508) (thermal_bridge_width 0.508))
+    (polygon
+      (pts
+        (xy 88.011 117.856) (xy 55.118 117.856) (xy 54.991 78.994) (xy 88.011 78.994)
+      )
+    )
+  )
 )
